File: eagle/NanoConnectionBoard.brd (EAGLE design)
At the start: 52.1 x 69.8 mm, 16 parts, among them J1 PINHD-1X121X12, Q1 600mA/40V, Q2 600mA/40V, Q3 FDN340P

Commit message: updated
Routing:
- net 3V3: track 8.67 -> 2.54 mm
Changed lines of the file:
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@@
 <contactref element="JP3" pad="2"/>
 <wire x1="-16.51" y1="5.08" x2="-13.97" y2="5.08" width="0.254" layer="1"/>
-<wire x1="-13.97" y1="5.08" x2="-11.43" y2="5.08" width="0.254" layer="1"/>
-<wire x1="-11.43" y1="5.08" x2="-8.89" y2="7.62" width="0.254" layer="1"/>
 </signal>
 <signal name="REF">
