File: eagle/OneBoard.sch (EAGLE design)
At the start: 29 parts

Commit message: updated
Parts:
- removed JP1: PINHD-1X12-FEMALE, Pat Sonstiges:PINHD-1X12-FEMALE
- added LSP1, LSP2: LSP11, solpad:LSP11
- added POWERBOOST: ADAFRUIT_POWERBOOST_1000C, My Breakout Boards:ADAFRUIT_POWERBOOST_1000C
- added RESET: TACTILE_BUTTON_6X6X9.5, Pat Sonstiges:TACTILE_BUTTON_6X6X9.5
- added SW1: (no value), Seeed-Switch:DIP-TOGGLE-SWITCH-2CH-(2X3P-2.54)
- added U$7: ARDUINO-NANO, My Boards:ARDUINO-NANO
- renumbered U$1 to DISPLAY, U$2 to RTC
Connections:
- new net 3V3: U$7.3V3
- new net A6: U$7.A6
- new net A7: U$7.A7
- new net BAT+: LSP1.MP, SW1.CH1A, SW1.CH2A
- new net D10: U$7.D10
- new net D11: U$7.D11
- new net D12: U$7.D12
- new net D13: U$7.D13
- new net D2: U$7.D2
- new net D3: U$7.D3
- new net D4: U$7.D4
- new net D6: U$7.D6
- new net D7: U$7.D7
- new net D8: U$7.D8
- new net D9: U$7.D9
- new net MISO: U$7.MISO
- new net MOSI: U$7.MOSI
- new net N$1: RTC.SDA1
- new net N$2: RTC.SCL1
- new net REF: U$7.REF
- new net RESET..: U$7.RESET..
- new net RST: RESET.2, RESET.4, U$7.RST
- new net RST.: U$7.RST.
- new net RX0: U$7.RX0
- new net SCK: U$7.SCK
- new net TX1: U$7.TX1
- new net VBAT: POWERBOOST.VBAT, SW1.COM1, SW1.COM2
- new net VIN_NANO: U$7.VIN
- new net VOUT: POWERBOOST.5V
- net 32K: no longer JP1.1
- net 5V: now also U$7.5V, U$7.5V.; no longer JP1.11
- net A0: now also C2.2, R5.2, S12.1, S12.3, S3.1, S3.3, S6.1, S6.3, S9.1, S9.3, U$7.A0; no longer JP1.4, U$4.S
- net A1: now also U$4.S, U$7.A1; no longer JP1.5
- net A2: now also U$7.A2; no longer JP1.6
- net A3: now also U$7.A3; no longer C2.2, JP1.7, R5.2, S12.1, S12.3, S3.1, S3.3, S6.1, S6.3, S9.1, S9.3
- net D5: now also U$7.D5; no longer JP1.10
- net GND: now also LSP2.MP, POWERBOOST.GND, RESET.1, RESET.3, U$7.GND, U$7.GND_; no longer JP1.12
- net GND_PWM: now also U$7.GND.; no longer JP1.3
- net SCL: now also U$7.A5; no longer JP1.8
- net SDA: now also U$7.A4; no longer JP1.9
- net SQW: no longer JP1.2
Other:
- moved on the sheet: C1, S+, U$5

Commit message: updated
Parts:
- R7: value 1k -> 470
Connections:
- removed net VOUT: POWERBOOST.5V
- net VIN_NANO: now also POWERBOOST.5V
Changed lines of the file:
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@@
 <part name="R5" library="rcl" library_urn="urn:adsk.eagle:library:334" deviceset="R-EU_" device="R0603" package3d_urn="urn:adsk.eagle:package:23555/2" value="1K"/>
 <part name="R6" library="rcl" library_urn="urn:adsk.eagle:library:334" deviceset="R-EU_" device="R0603" package3d_urn="urn:adsk.eagle:package:23555/2" value="820"/>
-<part name="R7" library="rcl" library_urn="urn:adsk.eagle:library:334" deviceset="R-EU_" device="R0603" package3d_urn="urn:adsk.eagle:package:23555/2" value="1k"/>
+<part name="R7" library="rcl" library_urn="urn:adsk.eagle:library:334" deviceset="R-EU_" device="R0603" package3d_urn="urn:adsk.eagle:package:23555/2" value="470"/>
 <part name="GND1" library="supply1" library_urn="urn:adsk.eagle:library:371" deviceset="GND" device=""/>
 <part name="C1" library="rcl" library_urn="urn:adsk.eagle:library:334" deviceset="C-EU" device="025-025X050" package3d_urn="urn:adsk.eagle:package:23629/2" value="x"/>
@@
 <label x="274.32" y="-71.12" size="1.778" layer="95" rot="R90"/>
 </segment>
+<segment>
+<pinref part="POWERBOOST" gate="G$1" pin="5V"/>
+<wire x1="233.68" y1="68.58" x2="243.84" y2="68.58" width="0.1524" layer="91"/>
+<label x="243.84" y="68.58" size="1.778" layer="95"/>
+</segment>
 </net>
 <net name="D12" class="0">
@@
 </segment>
 </net>
-<net name="VOUT" class="0">
-<segment>
-<pinref part="POWERBOOST" gate="G$1" pin="5V"/>
-<wire x1="233.68" y1="68.58" x2="243.84" y2="68.58" width="0.1524" layer="91"/>
-<label x="243.84" y="68.58" size="1.778" layer="95"/>
-</segment>
-</net>
